File: tec-1/hardware/kicad/tec-1-keybd.sch (KiCad schematic (older format))
At the start: 42 parts, among them J1 USB_C_Receptacle_USB2.0, SW10 SW_0, SW11 SW_7, SW12 SW_6, SW13 SW_5, SW14 SW_4, SW15 SW_B, SW16 SW_A, SW17 SW_9, SW18 SW_8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

Commit message: tec-1/hardware/kicad: progress checkin - add clock & 207 unrouted
Parts:
- C8: footprint (none) -> tec-1:CP_EIA-7343-31_Kemet-D; symbol tec-1:C -> tec-1:CP
- U8: footprint tec-1:DIP-18_W7.62mm_LongPads -> tec-1:DIP-20_W7.62mm_LongPads
Connections:
- net FTDI_D3: no longer U7.2 (DTR), U9.10 (FTDI_D4)
- net CC1: now reaches J1.A5 (CC1), R15.1
- net CC2: now reaches J1.B5 (CC2), R14.2
- net SHIELD: now reaches C7.2, J1.S1 (SHIELD), R13.1
- new net FTDI_D4: U7.2 (DTR), U9.10 (FTDI_D4)
Changed lines of the file:
@@
 $Descr A4 11693 8268
 encoding utf-8
-Sheet 2 3
+Sheet 3 3
 Title ""
 Date ""
@@
 FTDI_D3
 Text Label 4900 2500 0    50   ~ 0
-FTDI_D3
+FTDI_D4
 Text Label 4900 2600 0    50   ~ 0
 FTDI_D5
@@
 VBUS
 $Comp
-L tec-1:C C8
+L tec-1:CP C8
 U 1 1 61CAE9FC
 P 1350 1050
 F 0 "C8" H 1442 1096 50  0000 L CNN
 F 1 "100uF/10V" H 1442 1005 50  0000 L CNN
-F 2 "" H 1350 1050 50  0001 C CNN
+F 2 "tec-1:CP_EIA-7343-31_Kemet-D" H 1350 1050 50  0001 C CNN
 F 3 "~" H 1350 1050 50  0001 C CNN
 	1    1350 1050
@@
 L power:GND #PWR041
 U 1 1 61CAE9FD
-P 1350 1150
-F 0 "#PWR041" H 1350 900 50  0001 C CNN
-F 1 "GND" H 1355 977 50  0000 C CNN
-F 2 "" H 1350 1150 50  0001 C CNN
-F 3 "" H 1350 1150 50  0001 C CNN
-	1    1350 1150
+P 1350 1200
+F 0 "#PWR041" H 1350 950 50  0001 C CNN
+F 1 "GND" H 1355 1027 50  0000 C CNN
+F 2 "" H 1350 1200 50  0001 C CNN
+F 3 "" H 1350 1200 50  0001 C CNN
+	1    1350 1200
 	1    0    0    -1
 $EndComp
@@
 L power:+5V #PWR040
 U 1 1 607BF7BF
-P 1350 950
-F 0 "#PWR040" H 1350 800 50  0001 C CNN
-F 1 "+5V" H 1365 1123 50  0000 C CNN
-F 2 "" H 1350 950 50  0001 C CNN
-F 3 "" H 1350 950 50  0001 C CNN
-	1    1350 950
+P 1350 900
+F 0 "#PWR040" H 1350 750 50  0001 C CNN
+F 1 "+5V" H 1365 1073 50  0000 C CNN
+F 2 "" H 1350 900 50  0001 C CNN
+F 3 "" H 1350 900 50  0001 C CNN
+	1    1350 900
 	1    0    0    -1
 $EndComp
@@
 F 0 "U8" H 5000 7300 50  0000 C CNN
 F 1 "MM74C923" H 5500 7300 50  0000 C CNN
-F 2 "tec-1:DIP-18_W7.62mm_LongPads" H 5250 6650 50  0001 C CNN
+F 2 "tec-1:DIP-20_W7.62mm_LongPads" H 5250 6650 50  0001 C CNN
 F 3 "http://www.ti.com/lit/gpn/snMM74C923" H 5250 6650 50  0001 C CNN
 	1    5250 6650
@@
 Wire Wire Line
 	1800 6900 2400 6900
+Text Label 2000 1900 0    50   ~ 0
+CC1
+Text Label 2000 2000 0    50   ~ 0
+CC2
+Text Label 1100 3250 2    50   ~ 0
+SHIELD
 $EndSCHEMATC

Commit message: tec-1/hardware/kicad: routing complete, all DRC errors checked as ok
Parts:
- removed TP21, TP23: TestPoint, tec-1:TestPoint_Pad_D2.0mm, symbol tec-1:TestPoint
- added C22: 0.1uF/10V, tec-1:C_0805_2012Metric, symbol tec-1:C
- added D3: LED, tec-1:LED_0805_2012Metric, symbol tec-1:LED
- added R48: 1k, tec-1:R_0805_2012Metric, symbol tec-1:R
Connections:
- net +5V: now also C22.1, D3.2 (A)
- net D0: now also U9.20 (D0); no longer U9.19 (~NMI)
- net D1: now also U9.21 (D1); no longer U9.20 (D0)
- net D2: now also U9.23 (D2); no longer U9.21 (D1)
- net D3: now also U9.24 (D3); no longer U9.23 (D2)
- net D4: now also U9.25 (D4); no longer U9.24 (D3)
- net D5: now also U9.26 (D5); no longer U9.25 (D4)
- net GND: now also C22.2, R48.2
- net ~C923_OE: now also U9.18 (~C923_OE); no longer U9.17 (NC17)
- net ~NMI: now also U9.19 (~NMI); no longer U9.18 (~C923_OE)
- net ~SHIFT_KEY: now also U9.4 (~SHIFTKEY); no longer U9.15 (NC15)
- net at U9.2 (~FTDI_WR): now also U7.23 (CBUS0); no longer U9.26 (D5)
- new net: D3.1 (K), R48.1
- no-connect marks 9 -> 14
Changed lines of the file:
@@
 NoConn ~ 5500 3100
 NoConn ~ 5600 3100
-NoConn ~ 6050 3100
-NoConn ~ 6150 3100
+NoConn ~ 5700 3100
+NoConn ~ 5900 3100
 $Comp
 L power:GND #PWR057
@@
 	1    0    0    -1
 $EndComp
+Text Label 6450 2800 0    50   ~ 0
+D5
+Text Label 6450 2300 0    50   ~ 0
+D0
+Text Label 6450 2400 0    50   ~ 0
+D1
+Text Label 6450 2500 0    50   ~ 0
+D2
+Text Label 6450 2600 0    50   ~ 0
+D3
 Text Label 6450 2700 0    50   ~ 0
-D5
-Text Label 6450 2200 0    50   ~ 0
-D0
-Text Label 6450 2300 0    50   ~ 0
-D1
-Text Label 6450 2400 0    50   ~ 0
-D2
-Text Label 6450 2500 0    50   ~ 0
-D3
-Text Label 6450 2600 0    50   ~ 0
 D4
-Wire Wire Line
-	6350 2800 7050 2800
-Wire Wire Line
-	7050 2800 7050 1250
-Wire Wire Line
-	7050 1250 5200 1250
-Wire Wire Line
-	5200 1250 5200 1800
-Wire Wire Line
-	5200 1800 5300 1800
 Text Label 6450 1900 0    50   ~ 0
 KEYBD_CS
-Text Label 6450 2100 0    50   ~ 0
+Text Label 6450 2200 0    50   ~ 0
 ~NMI
 $Comp
@@
 Wire Wire Line
 	4800 3100 4850 3100
-Wire Wire Line
-	4850 3100 4850 2000
-Wire Wire Line
-	4850 2000 5300 2000
 Text Label 4900 2100 0    50   ~ 0
 FTDI_D0
@@
 	1    0    0    -1
 $EndComp
-Text Label 6450 2000 0    50   ~ 0
+Text Label 6450 2100 0    50   ~ 0
 ~C923_OE
 Text Label 5850 6850 0    50   ~ 0
@@
 	3600 6550 3700 6550
 $Comp
-L power:PWR_FLAG #FLG02
-U 1 1 607DDD0D
-P 2000 750
-F 0 "#FLG02" H 2000 825 50  0001 C CNN
-F 1 "PWR_FLAG" V 2000 878 50  0000 L CNN
-F 2 "" H 2000 750 50  0001 C CNN
-F 3 "~" H 2000 750 50  0001 C CNN
-	1    2000 750
-	0    1    1    0
-$EndComp
-Connection ~ 2000 750
-$Comp
 L power:PWR_FLAG #FLG03
 U 1 1 607DE749
@@
 	6350 1900 6450 1900
 Wire Wire Line
-	6350 2000 6450 2000
-Wire Wire Line
 	6350 2100 6450 2100
 Wire Wire Line
@@
 Wire Wire Line
 	6350 2700 6450 2700
+Wire Wire Line
+	6350 2800 6450 2800
 $Comp
 L tec-1:SW_SPST SW2
@@
 ~SHIFT_KEY
 Connection ~ 1000 5300
-Text Label 6450 1800 0    50   ~ 0
-~SHIFT_KEY
-Wire Wire Line
-	6350 1800 6450 1800
 Wire Wire Line
 	10400 3450 10300 3450
@@
 D4
 $Comp
+L tec-1:TestPoint TP22
+U 1 1 615B77A2
+P 5050 3500
+F 0 "TP22" H 4992 3572 50  0000 R CNN
+F 1 "TestPoint" H 4992 3617 50  0001 R CNN
+F 2 "tec-1:TestPoint_Pad_D2.0mm" H 5250 3500 50  0001 C CNN
+F 3 "~" H 5250 3500 50  0001 C CNN
+	1    5050 3500
+	-1   0    0    1
+$EndComp
+Wire Wire Line
+	4800 3400 5050 3400
+Wire Wire Line
+	5050 3400 5050 3500
+Wire Wire Line
+	1200 6900 1800 6900
+Wire Wire Line
+	1800 6750 1800 6900
+Connection ~ 1800 6900
+Wire Wire Line
+	1800 6900 2400 6900
+Text Label 2000 1900 0    50   ~ 0
+CC1
+Text Label 2000 2000 0    50   ~ 0
+CC2
+Text Label 1100 3250 2    50   ~ 0
+SHIELD
+$Comp
+L tec-1:C C22
+U 1 1 60749591
+P 4350 1300
+F 0 "C22" H 4442 1346 50  0000 L CNN
+F 1 "0.1uF/10V" H 4442 1255 50  0000 L CNN
+F 2 "tec-1:C_0805_2012Metric" H 4350 1300 50  0001 C CNN
+F 3 "~" H 4350 1300 50  0001 C CNN
+	1    4350 1300
+	1    0    0    -1
+$EndComp
+$Comp
+L power:GND #PWR0132
+U 1 1 6074997B
+P 4350 1400
+F 0 "#PWR0132" H 4350 1150 50  0001 C CNN
+F 1 "GND" H 4355 1227 50  0000 C CNN
+F 2 "" H 4350 1400 50  0001 C CNN
+F 3 "" H 4350 1400 50  0001 C CNN
+	1    4350 1400
+	1    0    0    -1
+$EndComp
+$Comp
+L power:+5V #PWR0133
+U 1 1 60749985
+P 4350 1200
+F 0 "#PWR0133" H 4350 1050 50  0001 C CNN
+F 1 "+5V" H 4365 1373 50  0000 C CNN
+F 2 "" H 4350 1200 50  0001 C CNN
+F 3 "" H 4350 1200 50  0001 C CNN
+	1    4350 1200
+	1    0    0    -1
+$EndComp
+Wire Wire Line
+	4800 3200 5250 3200
+$Comp
 L tec-1:TestPoint TP24
 U 1 1 615B6A1A
@@
 	-1   0    0    1
 $EndComp
-$Comp
-L tec-1:TestPoint TP23
-U 1 1 615B740B
-P 5150 3350
-F 0 "TP23" H 5092 3422 50  0000 R CNN
-F 1 "TestPoint" H 5092 3467 50  0001 R CNN
-F 2 "tec-1:TestPoint_Pad_D2.0mm" H 5350 3350 50  0001 C CNN
-F 3 "~" H 5350 3350 50  0001 C CNN
-	1    5150 3350
-	-1   0    0    1
-$EndComp
-$Comp
-L tec-1:TestPoint TP22
-U 1 1 615B77A2
-P 5050 3500
-F 0 "TP22" H 4992 3572 50  0000 R CNN
-F 1 "TestPoint" H 4992 3617 50  0001 R CNN
-F 2 "tec-1:TestPoint_Pad_D2.0mm" H 5250 3500 50  0001 C CNN
-F 3 "~" H 5250 3500 50  0001 C CNN
-	1    5050 3500
-	-1   0    0    1
-$EndComp
-$Comp
-L tec-1:TestPoint TP21
-U 1 1 615B7B90
-P 4950 3650
-F 0 "TP21" H 4892 3722 50  0000 R CNN
-F 1 "TestPoint" H 4892 3767 50  0001 R CNN
-F 2 "tec-1:TestPoint_Pad_D2.0mm" H 5150 3650 50  0001 C CNN
-F 3 "~" H 5150 3650 50  0001 C CNN
-	1    4950 3650
-	-1   0    0    1
-$EndComp
-Wire Wire Line
-	4800 3200 5250 3200
-Wire Wire Line
-	5150 3350 5150 3300
-Wire Wire Line
-	5150 3300 4800 3300
-Wire Wire Line
-	4800 3400 5050 3400
-Wire Wire Line
-	5050 3400 5050 3500
-Wire Wire Line
-	4800 3500 4950 3500
-Wire Wire Line
-	4950 3500 4950 3650
-Wire Wire Line
-	1200 6900 1800 6900
-Wire Wire Line
-	1800 6750 1800 6900
-Connection ~ 1800 6900
-Wire Wire Line
-	1800 6900 2400 6900
-Text Label 2000 1900 0    50   ~ 0
-CC1
-Text Label 2000 2000 0    50   ~ 0
-CC2
-Text Label 1100 3250 2    50   ~ 0
-SHIELD
+NoConn ~ 4800 3300
+NoConn ~ 4800 3500
+$Comp
+L power:+5V #PWR?
+U 1 1 60986F67
+P 2450 750
+AR Path="/608A5BD6/60986F67" Ref="#PWR?"  Part="1"
+AR Path="/60617BAD/60986F67" Ref="#PWR0134"  Part="1"
+F 0 "#PWR0134" H 2450 600 50  0001 C CNN
+F 1 "+5V" H 2465 923 50  0000 C CNN
+F 2 "" H 2450 750 50  0001 C CNN
+F 3 "" H 2450 750 50  0001 C CNN
+	1    2450 750
+	-1   0    0    -1
+$EndComp
+$Comp
+L tec-1:LED D?
+U 1 1 60986F6D
+P 2450 900
+AR Path="/608A5BD6/60986F6D" Ref="D?"  Part="1"
+AR Path="/60617BAD/60986F6D" Ref="D3"  Part="1"
+F 0 "D3" V 2489 782 50  0000 R CNN
+F 1 "LED" V 2398 782 50  0000 R CNN
+F 2 "tec-1:LED_0805_2012Metric" H 2450 900 50  0001 C CNN
+F 3 "~" H 2450 900 50  0001 C CNN
+	1    2450 900
+	0    -1   -1   0
+$EndComp
+$Comp
+L tec-1:R R?
+U 1 1 60986F73
+P 2450 1250
+AR Path="/608A5BD6/60986F73" Ref="R?"  Part="1"
+AR Path="/60617BAD/60986F73" Ref="R48"  Part="1"
+F 0 "R48" V 2450 1200 50  0000 L CNN
+F 1 "1k" H 2509 1205 50  0001 L CNN
+F 2 "tec-1:R_0805_2012Metric" H 2450 1250 50  0001 C CNN
+F 3 "~" H 2450 1250 50  0001 C CNN
+	1    2450 1250
+	1    0    0    -1
+$EndComp
+Wire Wire Line
+	2450 1050 2450 1150
+$Comp
+L power:GND #PWR0135
+U 1 1 6098FDA7
+P 2450 1350
+F 0 "#PWR0135" H 2450 1100 50  0001 C CNN
+F 1 "GND" H 2455 1177 50  0000 C CNN
+F 2 "" H 2450 1350 50  0001 C CNN
+F 3 "" H 2450 1350 50  0001 C CNN
+	1    2450 1350
+	1    0    0    -1
+$EndComp
+NoConn ~ 6350 2900
+Wire Wire Line
+	4850 1800 5300 1800
+Wire Wire Line
+	4850 1800 4850 3100
+Text Label 5300 2000 2    50   ~ 0
+~SHIFT_KEY
+NoConn ~ 6350 2000
+NoConn ~ 6350 1800
 $EndSCHEMATC
